File: Apollo4_SE_Left_V3.kicad_pcb (KiCad board)
At the start: 6 copper layers, 0 parts

Commit message: [PCB] See Changelog for details
Parts:
- added ?: , , F.Cu at (110.6, 100.1)
- added ?: , , F.Cu at (111.8, 100.0)
- added ? (x2): , , B.Cu at (111.9, 90.9)
- added BM1: Conn_01x01_MountingPin, apollo4_SE:Solderwire_8_4, F.Cu at (107.4, 100.6)
- added BP1: Conn_01x01_MountingPin, apollo4_SE:Solderwire_8_4, F.Cu at (106.1, 100.6)
- added C1: 6pF, apollo4_SE:SMT_0201_0603Metric, B.Cu at (103.3, 98.0)
- added C10: 2.2uF, apollo4_SE:SMT_0201_0603Metric, F.Cu at (104.8, 93.5)
- added C11: 2.2uF, apollo4_SE:SMT_0201_0603Metric, F.Cu at (106.7, 94.7)
- added C12: 2.2uF, apollo4_SE:SMT_0201_0603Metric, F.Cu at (106.8, 93.4)
- added C13: 2.2uF, apollo4_SE:SMT_0201_0603Metric, F.Cu at (106.8, 94.1)
- added C14: 2.2uF, apollo4_SE:SMT_0201_0603Metric, F.Cu at (103.0, 91.6)
- added C15: 2.2uF, apollo4_SE:SMT_0201_0603Metric, F.Cu at (101.5, 91.6)
- added C16: 4.7uF, apollo4_SE:SMT_0201_0603Metric, F.Cu at (98.7, 97.3)
- added C17: 1uF, apollo4_SE:SMT_0201_0603Metric, F.Cu at (100.7, 91.6)
- added C18: 6pF, apollo4_SE:SMT_0201_0603Metric, B.Cu at (105.2, 94.1)
- added C19: 0.1uF, apollo4_SE:SMT_0201_0603Metric, F.Cu at (115.6, 96.8)
- added C2: 6pF, apollo4_SE:SMT_0201_0603Metric, B.Cu at (102.5, 97.4)
- added C20: 10uF, apollo4_SE:SMT_0402_1005Metric, F.Cu at (109.4, 97.2)
- added C21: 0.1uF, apollo4_SE:SMT_0201_0603Metric, F.Cu at (110.2, 97.3)
- added C22: 1uF, apollo4_SE:SMT_0201_0603Metric, F.Cu at (93.1, 99.1)
- added C23: 1uF, apollo4_SE:SMT_0201_0603Metric, F.Cu at (93.5, 96.9)
- added C24: 1uF, apollo4_SE:SMT_0201_0603Metric, F.Cu at (104.4, 98.5)
- added C25: 1uF, apollo4_SE:SMT_0201_0603Metric, F.Cu at (106.5, 97.6)
- added C26: 6pF, apollo4_SE:SMT_0201_0603Metric, F.Cu at (112.7, 96.0)
- added C27: 1.5pF, apollo4_SE:SMT_0201_0603Metric, F.Cu at (98.8, 91.6)
- added C3: 6pF, apollo4_SE:SMT_0201_0603Metric, B.Cu at (105.3, 95.3)
- added C4: 1uF, apollo4_SE:SMT_0201_0603Metric, F.Cu at (103.6, 91.6)
- added C5: 1uF, apollo4_SE:SMT_0201_0603Metric, F.Cu at (98.4, 96.4)
- added C6: 1uF, apollo4_SE:SMT_0201_0603Metric, F.Cu at (98.4, 95.7)
- added C7: 1uF, apollo4_SE:SMT_0201_0603Metric, F.Cu at (102.0, 91.6)
- added C8: 2.2uF, apollo4_SE:SMT_0201_0603Metric, F.Cu at (104.8, 96.8)
- added C9: 2.2uF, apollo4_SE:SMT_0201_0603Metric, F.Cu at (101.5, 98.0)
- added J1: TC2030-IDC, TC2030:TC2030_THL_PINS, F.Cu at (112.5, 92.8)
- added J2: MM8030-2610RJ3, apollo4_SE:MURATA_MM8030-2610RJ3, B.Cu at (98.8, 91.3)
- added JP1: SolderJumper_2_Bridged, Solder_Pad_Tiny:SolderJumper-Tiny_CLOSED, B.Cu at (112.6, 99.2)
- added JP2: SolderJumper_2_Open, Solder_Pad_Tiny:SolderJumper-Tiny_OPEN, B.Cu at (113.2, 99.6)
- added JP3: SolderJumper_2_Bridged, Solder_Pad_Tiny:SolderJumper-Tiny_CLOSED, B.Cu at (98.4, 98.5)
- added L1: AMCA31-2R450G-S1F-T3, apollo4_SE:ANTC3216X140N, F.Cu at (93.2, 92.2)
- added L2: DFE201210U-2R2M=P2 (verified), DFE201210U-2R2M=P2:IND_DFE201210U-2R2M=P2_MUR, F.Cu at (105.7, 92.0)
- added L3: MLF1005G1R0KT000, apollo4_SE:LQW15CNR20J00B, F.Cu at (100.4, 97.8)
- added L4: 2.2nH, apollo4_SE:INDC0603X33N, F.Cu at (99.7, 91.6)
- added L5: 2.0 nH, apollo4_SE:IND_LQP03HQ2N0B02D, F.Cu at (98.8, 93.0)
- added LED1: XL-0201UWC, LED_SMD:LED_0201_0603Metric, F.Cu at (96.6, 99.2)
- added LED2: XL-0201SURC, LED_SMD:LED_0201_0603Metric, F.Cu at (96.6, 99.9)
- added LED3: XL-0201SURC, LED_SMD:LED_0201_0603Metric, F.Cu at (109.7, 94.4)
- added LED4: XL-0201UGC, LED_SMD:LED_0201_0603Metric, F.Cu at (109.7, 95.1)
- added LED5: XL-0201UBC, LED_SMD:LED_0201_0603Metric, F.Cu at (109.7, 95.9)
- added MIC1: MMICT390200012, MMICT5837:MIC_MMICT5837-00-012, F.Cu at (114.6, 98.2)
- added R1: 2.2K, apollo4_SE:SMT_0201_0603Metric, F.Cu at (108.7, 97.3)
- added R10: 100K, apollo4_SE:SMT_0201_0603Metric, F.Cu at (105.0, 98.5)
- added R11: 100K, apollo4_SE:SMT_0201_0603Metric, F.Cu at (109.7, 93.1)
- added R12: 150, apollo4_SE:SMT_0201_0603Metric, F.Cu at (109.7, 93.8)
- added R13: 150, apollo4_SE:SMT_0201_0603Metric, F.Cu at (107.7, 95.3)
- added R14: 150, apollo4_SE:SMT_0201_0603Metric, F.Cu at (108.3, 95.9)
- added R15: 4.7K, apollo4_SE:SMT_0201_0603Metric, F.Cu at (113.3, 96.0)
- added R2: 2.2K, apollo4_SE:SMT_0201_0603Metric, F.Cu at (107.9, 97.3)
- added R3: 30, apollo4_SE:SMT_0201_0603Metric, F.Cu at (105.2, 97.6)
- added R4: 30, apollo4_SE:SMT_0201_0603Metric, F.Cu at (111.4, 97.1)
- added R5: 30, apollo4_SE:SMT_0201_0603Metric, F.Cu at (106.2, 96.8)
- added R6: 200K, apollo4_SE:SMT_0201_0603Metric, F.Cu at (94.9, 96.8)
- added R7: 2.4K, apollo4_SE:SMT_0201_0603Metric, F.Cu at (93.1, 97.9)
- added R8: 150, apollo4_SE:SMT_0201_0603Metric, F.Cu at (98.0, 99.1)
- added R9: 150, apollo4_SE:SMT_0201_0603Metric, F.Cu at (98.0, 99.9)
- added REF**: TestPoint_Pico, TestPoint:TestPoint_Pico, B.Cu at (112.9, 97.6)
- added REF**: TestPoint_Pico, TestPoint:TestPoint_Pico, B.Cu at (98.5, 95.1)
- added REF**: TestPoint_Pico, TestPoint:TestPoint_Pico, B.Cu at (113.8, 97.0)
- added S1: NANOT160AS, NANOT160AS:NANOT160AS, F.Cu at (111.3, 95.1)
- added U1: AMA4B2KL-KXR, apollo4_SE:AMA4B2KL-KXR, F.Cu at (101.6, 94.9)
- added U2: SSM6515BCBZRL7, SSM6515:SSM6515BCBZRL, F.Cu at (108.9, 98.8)
- added U3: TPB4056A20-DFGR, TPB4056A20:DFN2X2-8_TPK, F.Cu at (94.5, 98.7)
- added U4: TLV70718PDQNR, DQN:DQN0004A-MFG, F.Cu at (106.1, 98.5)
- added X1: LQW15AN9N7G80D, apollo4_SE:SMT_0402_1005Metric, F.Cu at (96.9, 92.7)
- added X2: SDCL1005C3N9STDF, apollo4_SE:SMT_0402_1005Metric, F.Cu at (97.8, 91.7)
- added Y1: SX16Y032000B61T001, apollo4_SE:XOSC_ABM12W_1.2x1.6, F.Cu at (102.8, 98.1)
- added Y2: ECS-.327-7-16-C-TR, AP510EVB:XTAL2-1P6X1P0-SM, F.Cu at (104.9, 94.7)
Routing:
- net REG_1.9V: track 0.00 -> 62.8 mm, vias 0 -> 22
- net GND: track 0.00 -> 52.2 mm, vias 0 -> 398
- net BAT+: track 0.00 -> 31.0 mm, vias 0 -> 6
- net SWCLK_GP20: track 0.00 -> 25.5 mm, vias 0 -> 4
- net I2S0_CLK: track 0.00 -> 17.8 mm, vias 0 -> 4
- net SWO_GP24: track 0.00 -> 17.4 mm, vias 0 -> 2
- net SWDIO_GP21: track 0.00 -> 15.2 mm, vias 0 -> 3
- net PDM0_CLK_GP50: track 0.00 -> 14.1 mm, vias 0 -> 2
- net nRST: track 0.00 -> 12.9 mm, vias 0 -> 4
- net BUTTON_0: track 0.00 -> 12.4 mm, vias 0 -> 2
- net PDM0_DATA_GP51: track 0.00 -> 11.1 mm, vias 0 -> 4
- net /MCU_Core/VDDBH: track 0.00 -> 11.0 mm, vias 0 -> 3
- net I2S0_DATA: track 0.00 -> 10.7 mm, vias 0 -> 2
- net IOM1_SDA: track 0.00 -> 10.6 mm, vias 0 -> 2
- net I2S0_WS: track 0.00 -> 9.10 mm, vias 0 -> 2
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- added copper zone on B.Cu, net GND
- added copper zone on F.Cu, net GND
Other:
- board outline added: 27.5 x 11.5 mm
- copper layers 6 -> 2
- rule pad_to_mask_clearance: 0.05 -> 0
- board text added: "+"
- board text added: "1"
- board text added: "5V"
- board text added: "6"
- board text added: "BAT"
- board text added: "L"
- board text added: "LDO EN"
- board text added: "PDM0_CLK"
- board text added: "PDM0_DATA"
- board text added: "PERSEV.ai"
- board text added: "R"
- board text added: "SPK"
- board text added: "TP 1V9"
- board text added: "V0.2 - 2026.1.29"
- board text added: "_"
- board text removed: "${ASSEMBLY_NOTES}"
- board text removed: "${FABRICATION_NOTES}"
- board text removed: "30°"
- board text removed: "3× 120°"
- board text removed: "All dimensions are in millimeters unless otherwise specified."
- board text removed: "Bottom View"
- board text removed: "Components"
- board text removed: "Drill Table"
- board text removed: "Impedance Table"
- board text removed: "Layer Stack Legend"
- board text removed: "Top View"
- board text removed: "X"
- board text removed: "Y"
