File: Apollo4_SE_Left_V3.kicad_sch (KiCad schematic)
At the start: 0 parts

Commit message: [PCB] See Changelog for details
Other:
- removed sheet Block Diagram
- removed sheet Power - Sequencing
- removed sheet Project Architecture
- removed sheet Revision History
- added sheet Antenna (antenna.kicad_sch)
- added sheet Audio (Audio.kicad_sch)
- added sheet MCU_Core (MCU_Core.kicad_sch)
- added sheet MCU_GPIO (MCU_GPIO.kicad_sch)
- added sheet Peripherals (Peripherals.kicad_sch)
- added sheet Power (Battery_Charger.kicad_sch)
- note added: "Back"
- note added: "Front"
- note added: "PERSEV.ai Speech Enhancement Ear Bud V0.2 01/24/2026"
- note added: "Schematics"
- note removed: "${BOARD_NAME}"
- note removed: "${RELEASE_DATE_NUM}"
- note removed: "${SHEET_NAME_10}"
- note removed: "${SHEET_NAME_11}"
- note removed: "${SHEET_NAME_12}"
- note removed: "${SHEET_NAME_13}"
- note removed: "${SHEET_NAME_14}"
- note removed: "${SHEET_NAME_15}"
- note removed: "${SHEET_NAME_16}"
- note removed: "${SHEET_NAME_17}"
- note removed: "${SHEET_NAME_18}"
- note removed: "${SHEET_NAME_19}"
- note removed: "${SHEET_NAME_1}"
- note removed: "${SHEET_NAME_20}"
- note removed: "${SHEET_NAME_21}"
- note removed: "${SHEET_NAME_22}"
- note removed: "${SHEET_NAME_23}"
- note removed: "${SHEET_NAME_24}"
- note removed: "${SHEET_NAME_25}"
- note removed: "${SHEET_NAME_26}"
- note removed: "${SHEET_NAME_27}"
- note removed: "${SHEET_NAME_28}"
- note removed: "${SHEET_NAME_29}"
- note removed: "${SHEET_NAME_2}"
- note removed: "${SHEET_NAME_30}"
- note removed: "${SHEET_NAME_31}"
- note removed: "${SHEET_NAME_32}"
- note removed: "${SHEET_NAME_33}"
- note removed: "${SHEET_NAME_34}"
- note removed: "${SHEET_NAME_35}"
- note removed: "${SHEET_NAME_36}"
- note removed: "${SHEET_NAME_37}"
- note removed: "${SHEET_NAME_38}"
- note removed: "${SHEET_NAME_39}"
- note removed: "${SHEET_NAME_3}"
- note removed: "${SHEET_NAME_40}"
- note removed: "${SHEET_NAME_4}"
- note removed: "${SHEET_NAME_5}"
- note removed: "${SHEET_NAME_6}"
- note removed: "${SHEET_NAME_7}"
- note removed: "${SHEET_NAME_8}"
- note removed: "${SHEET_NAME_9}"
- note removed: "1"
- note removed: "10"
- note removed: "11"
- note removed: "12"
- note removed: "13"
- note removed: "14"
- note removed: "15"
- note removed: "16"
- note removed: "17"
- note removed: "18"
- note removed: "19"
- note removed: "2"
- note removed: "20"
- note removed: "21"
- note removed: "22"
- note removed: "23"
- note removed: "24"
- note removed: "25"
- note removed: "26"
- note removed: "27"
- note removed: "28"
- note removed: "29"
- note removed: "3"
- note removed: "30"
- note removed: "31"
- note removed: "32"
- note removed: "33"
- note removed: "34"
- note removed: "35"
- note removed: "36"
- note removed: "37"
- note removed: "38"
- note removed: "39"
- note removed: "4"
- note removed: "40"
- note removed: "5"
- note removed: "6"
- note removed: "7"
- note removed: "8"
- note removed: "9"
- note removed: "BOTTOM VIEW"
- note removed: "CHECKED - There shouldn't be any mistakes. Contact the engineer if you find any."
- note removed: "Comment"
- note removed: "DESIGN CONSIDERATIONS"
- note removed: "DRAFT - Very early stage of schematic, ignore details."
- note removed: "Date: ${RELEASE_DATE}"
- note removed: "Index"
- note removed: "NOTES"
- note removed: "Not fitted components are marked as"
- note removed: "PRELIMINARY - Close to final schematic."
- note removed: "Page"
- note removed: "RELEASED - A board with this schematic has been sent to production."
- note removed: "Rev ${REVISION}"
- note removed: "TOP VIEW"
- note removed: "Variant: ${VARIANT}"
- company: ${COMPANY} -> (none)
- title: (none) -> Speech Enhancement Ear Bud
